File: kicad/interfaceboard/interfaceboard.kicad_pcb (KiCad board)
At the start: 2 copper layers, 194 parts, among them J1 HighSide Driver, J10 Interlock, J11 I2CEXT, J12 USB_LOG, J13 USB_CMD2, J14 USB_CMD1, J15 DB15_Female_MountingHoles, J16 DB15_Female_MountingHoles, J17 DB15_Female_MountingHoles, J18 DB15_Female_MountingHoles, J19 Screw_Terminal_01x02, J2 Interlock, J3 VCCCON, J4 ICSP, J5 Conn_02x05_Odd_Even, J6 GPIOEXT, J7 GNDCON, J8 Interlock, J9 Interlock, U1 ATmega2560-16A, U10 LM358, U11 MCP4822, U12 MCP4822, U13 MCP4822, U14 MCP4822, U15 PC817, U16 PC817, U17 PC817, U18 PC817, U19 PC817, U2 MCP3424, U20 PC817, U21 PC817, U22 PC817, U23 AC-05-3, U3 MCP3424, U4 CP2102N-Axx-xQFN28, U5 CP2102N-Axx-xQFN28, U6 CP2102N-Axx-xQFN28, U7 LM358, U8 LM358, U9 LM358, Y1 16MHz

Commit message: Continue place and route, minor fixes
Parts:
- J10: value Interlock -> USART3
- J8: value Interlock -> USART1
- J9: value Interlock -> USART2
- moved J12 143.3 mm to (242.5, 127.9), turned to -90 degrees
- moved J10 142.5 mm to (229.8, 115.6)
- moved R27 136.1 mm to (100.3, 51.4), turned to 90 degrees
- moved D11 134.9 mm to (248.9, 110.5), turned to 180 degrees
- moved D13 129.7 mm to (218.7, 110.5), turned to 180 degrees
- moved R51 126.0 mm to (68.6, 48.3), turned to 90 degrees
- moved J14 125.2 mm to (186.6, 127.9), turned to -90 degrees
- moved C6 124.7 mm to (194.3, 62.2), turned to -90 degrees
- moved R76 122.8 mm to (72.4, 44.5), turned to 90 degrees
- moved C13 117.9 mm to (240.0, 91.4)
- moved C17 115.3 mm to (216.2, 90.2)
- moved R55 115.1 mm to (68.6, 44.5), turned to 90 degrees
- moved R58 113.4 mm to (72.4, 48.3), turned to 90 degrees
- moved R77 112.5 mm to (76.2, 44.5), turned to 90 degrees
- moved R34 109.5 mm to (216.2, 54.6)
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Connections:
- J16 pad 1: /CC_{1} -> /CC_{3}
- J16 pad 11: /V_{mon} -> V_{mon,3}
- J16 pad 12: UNIT_{ON,1} -> UNIT_{ON,3}
- J16 pad 15: /I_{set,1} -> /I_{set,3}
- J16 pad 2: /CV_{1} -> /CV_{3}
- J16 pad 3: /I_{mon} -> I_{mon,3}
- J16 pad 7: POL_{set,1} -> POL_{set,3}
- J16 pad 8: /V_{set,1} -> /V_{set,3}
- J17 pad 1: /CC_{1} -> /CC_{2}
- J17 pad 11: /V_{mon} -> V_{mon,2}
- J17 pad 12: UNIT_{ON,1} -> UNIT_{ON,2}
- J17 pad 15: /I_{set,1} -> /I_{set,2}
- J17 pad 2: /CV_{1} -> /CV_{2}
- J17 pad 3: /I_{mon} -> I_{mon,2}
- J17 pad 7: POL_{set,1} -> POL_{set,2}
- J17 pad 8: /V_{set,1} -> /V_{set,2}
- J18 pad 1: /CC_{1} -> /CC_{4}
- J18 pad 11: /V_{mon} -> V_{mon,4}
- J18 pad 12: UNIT_{ON,1} -> UNIT_{ON,4}
- J18 pad 15: /I_{set,1} -> /I_{set,4}
- J18 pad 2: /CV_{1} -> /CV_{4}
- J18 pad 3: /I_{mon} -> I_{mon,4}
- J18 pad 7: POL_{set,1} -> POL_{set,4}
- J18 pad 8: /V_{set,1} -> /V_{set,4}
- R45 pad 2: /V_{set,1} -> /V_{set,3}
- R46 pad 2: /I_{set,1} -> /I_{set,3}
- R47 pad 2: /V_{set,1} -> /V_{set,2}
- R48 pad 2: /I_{set,1} -> /I_{set,2}
- R49 pad 2: /V_{set,1} -> /V_{set,4}
- R50 pad 2: /I_{set,1} -> /I_{set,4}
- R57 pad 2: /CC_{1} -> /CC_{3}
- R61 pad 2: /CC_{1} -> /CC_{2}
- R67 pad 2: /CC_{1} -> /CC_{4}
- R81 pad 2: /CV_{1} -> /CV_{3}
- R82 pad 2: /I_{mon} -> I_{mon,3}
- R83 pad 2: /V_{mon} -> V_{mon,3}
- R84 pad 2: /CV_{1} -> /CV_{2}
- R85 pad 2: /I_{mon} -> I_{mon,2}
- R86 pad 2: /V_{mon} -> V_{mon,2}
- R88 pad 2: /CV_{1} -> /CV_{4}
- R89 pad 2: /I_{mon} -> I_{mon,4}
- R90 pad 2: /V_{mon} -> V_{mon,4}
- U1 pad 65: ~{USB_{RST,1}} -> unconnected-(U1-Pad65)
- U1 pad 66: ~{USB_{RST,2}} -> unconnected-(U1-Pad66)
- U1 pad 67: ~{USB_{RST,3}} -> unconnected-(U1-Pad67)
- U10 pad 1: /V_{set,1} -> /V_{set,4}
- U10 pad 7: /I_{set,1} -> /I_{set,4}
- U17 pad 4: POL_{set,1} -> POL_{set,3}
- U18 pad 4: UNIT_{ON,1} -> UNIT_{ON,3}
- U19 pad 4: POL_{set,1} -> POL_{set,2}
- U20 pad 4: UNIT_{ON,1} -> UNIT_{ON,2}
- U21 pad 4: POL_{set,1} -> POL_{set,4}
- U22 pad 4: UNIT_{ON,1} -> UNIT_{ON,4}
- U8 pad 1: /V_{set,1} -> /V_{set,3}
- U8 pad 7: /I_{set,1} -> /I_{set,3}
- U9 pad 1: /V_{set,1} -> /V_{set,2}
- U9 pad 7: /I_{set,1} -> /I_{set,2}
Routing:
- net GND: track 0.00 -> 700.8 mm, vias 0 -> 3
- net +5V: track 0.00 -> 192.6 mm, vias 0 -> 6
- net SCL: track 0.00 -> 151.2 mm, vias 0 -> 4
- net SDA: track 0.00 -> 145.1 mm, vias 0 -> 6
- net ~{RESET}: track 0.00 -> 119.5 mm, vias 0 -> 3
- net I_{mon,3}: track 0.00 -> 55.5 mm, vias 0 -> 4
- net V_{mon,3}: track 0.00 -> 51.1 mm, vias 0 -> 4
- net CC3: track 0.00 -> 44.7 mm
- net CV3: track 0.00 -> 44.3 mm
- net /V_{set,2}: track 0.00 -> 34.0 mm
- net /I_{set,2}: track 0.00 -> 33.8 mm
- net /V_{set,1}: track 0.00 -> 32.8 mm
- net /I_{set,1}: track 0.00 -> 32.5 mm
- net /I_{set,4}: track 0.00 -> 32.5 mm
- net V_{mon,2}: track 0.00 -> 32.5 mm
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Other:
- board outline added: 186.1 x 125.7 mm
