File: kicad/interfaceboard/interfaceboard.kicad_sch (KiCad schematic)
At the start: 133 parts

Commit message: Finished schematic
Parts:
- added C? (x3): 1.0uF, symbol Device:C_Small
- added C? (x6): 0.1uF, symbol Device:C_Small
- added C? (x3): 4.7uF, symbol Device:C_Polarized_Small
- added D? (x11): LED, symbol Device:LED
- added D? (x3): SP0503BAHT, Package_TO_SOT_SMD:SOT-143, symbol Power_Protection:SP0503BAHT
- added J?: GPIOEXT, symbol Connector_Generic:Conn_02x16_Counter_Clockwise
- added J?: Conn_02x05_Odd_Even, symbol Connector_Generic:Conn_02x05_Odd_Even
- added J?: Interlock, symbol Connector:Screw_Terminal_01x02
- added J?: USB_CMD2, symbol Connector:USB_B
- added J?: USB_CMD1, symbol Connector:USB_B
- added J?: VCCCON, symbol Connector_Generic:Conn_02x16_Counter_Clockwise
- added J?: USB_LOG, symbol Connector:USB_B
- added J?: GNDCON, symbol Connector_Generic:Conn_02x16_Counter_Clockwise
- added J?: I2CEXT, symbol Connector_Generic:Conn_02x04_Counter_Clockwise
- added JP? (x3): RSTEN, symbol Jumper:Jumper_2_Bridged
- added L?: 10uH, symbol Device:L_Small
- added R?: 1M, symbol Device:R_Small
- added R? (x6): 1k, symbol Device:R_Small
- added R? (x4): 10k, symbol Device:R_Small
- added R? (x3): 24k, symbol Device:R_Small
- added R? (x3): 47k, symbol Device:R_Small
- added R? (x5): 390R, symbol Device:R_Small
- added U? (x3): CP2102N-Axx-xQFN28, Package_DFN_QFN:QFN-28-1EP_5x5mm_P0.5mm_EP3.35x3.35mm, symbol Interface_USB:CP2102N-Axx-xQFN28
- D?: value LED -> LED_{PWR}
- R? (x9): value R_Small -> 390R
Connections:
- net +5V: now also C?.1, C?.1, C?.1, C?.1, C?.1, C?.1, J?.1 (Pin_1), J?.1 (Pin_1), J?.1 (Pin_1), J?.10 (Pin_10), J?.11 (Pin_11), J?.12 (Pin_12), J?.13 (Pin_13), J?.14 (Pin_14), J?.15 (Pin_15), J?.16 (Pin_16), J?.17 (Pin_17), J?.18 (Pin_18), J?.19 (Pin_19), J?.2 (Pin_2), J?.20 (Pin_20), J?.21 (Pin_21), J?.22 (Pin_22), J?.23 (Pin_23), J?.24 (Pin_24), J?.25 (Pin_25), J?.26 (Pin_26), J?.27 (Pin_27), J?.28 (Pin_28), J?.29 (Pin_29), J?.3 (Pin_3), J?.30 (Pin_30), J?.31 (Pin_31), J?.32 (Pin_32), J?.4 (Pin_4), J?.5 (Pin_5), J?.6 (Pin_6), J?.7 (Pin_7), J?.8 (Pin_8), J?.8 (Pin_8), J?.9 (Pin_9), L?.1, R?.2, U?.7 (VREGIN), U?.7 (VREGIN), U?.7 (VREGIN); no longer U?.100 (AVCC)
- net GND: now also C?.2, C?.2, C?.2, C?.2, C?.2, C?.2, D?.1 (A), D?.1 (A), D?.1 (A), D?.1 (K), D?.1 (K), D?.1 (K), D?.1 (K), D?.1 (K), D?.1 (K), D?.1 (K), D?.1 (K), D?.1 (K), D?.1 (K), D?.1 (K), J?.1 (Pin_1), J?.10 (Pin_10), J?.11 (Pin_11), J?.12 (Pin_12), J?.13 (Pin_13), J?.14 (Pin_14), J?.15 (Pin_15), J?.16 (Pin_16), J?.17 (Pin_17), J?.18 (Pin_18), J?.19 (Pin_19), J?.2 (Pin_2), J?.20 (Pin_20), J?.21 (Pin_21), J?.22 (Pin_22), J?.23 (Pin_23), J?.24 (Pin_24), J?.25 (Pin_25), J?.26 (Pin_26), J?.27 (Pin_27), J?.28 (Pin_28), J?.29 (Pin_29), J?.3 (Pin_3), J?.3 (Pin_3), J?.30 (Pin_30), J?.31 (Pin_31), J?.32 (Pin_32), J?.4 (GND), J?.4 (GND), J?.4 (GND), J?.4 (Pin_4), J?.4 (Pin_4), J?.5 (Pin_5), J?.5 (Pin_5), J?.5 (Pin_5), J?.5 (Shield), J?.5 (Shield), J?.5 (Shield), J?.6 (Pin_6), J?.7 (Pin_7), J?.8 (Pin_8), J?.9 (Pin_9), J?.9 (Pin_9), R?.1, R?.1, R?.1, R?.2, R?.2, R?.2, R?.2, U?.29 (GND), U?.29 (GND), U?.29 (GND), U?.3 (GND), U?.3 (GND), U?.3 (GND)
- net SCL: now also J?.2 (Pin_2), J?.7 (Pin_7)
- net SDA: now also J?.3 (Pin_3), J?.6 (Pin_6)
- net ~{CS_{PSU1}}: now also U?.36 (PL1)
- net ~{CS_{PSU2}}: now also U?.37 (PL2)
- net ~{CS_{PSU3}}: now also U?.38 (PL3)
- net ~{CS_{PSU4}}: now also U?.39 (PL4)
- net ~{LDAC}: now also U?.35 (PL0)
- net ~{RESET}: now also J?.10 (Pin_10), JP?.2 (B), JP?.2 (B), JP?.2 (B)
- net PH5: now reaches U?.1 (PG5)
- net PH5: now also U?.17 (PH5), J?.15 (Pin_15), J?.24 (Pin_24)
- net PH2: now reaches U?.14 (PH2)
- net PH2: now also U?.70 (PG2), J?.12 (Pin_12), J?.21 (Pin_21)
- net PH3: now reaches U?.15 (PH3)
- net PH3: now also U?.28 (PG3), J?.13 (Pin_13), J?.22 (Pin_22)
- net PH4: now reaches U?.16 (PH4)
- net PH4: now also U?.29 (PG4), J?.14 (Pin_14), J?.23 (Pin_23)
- net PH6: now reaches U?.18 (PH6)
- net PH6: now also J?.16 (Pin_16)
- net USB_{1,RX}: now reaches U?.2 (PE0)
- net USB_{1,RX}: now also U?.63 (PJ0), U?.26 (TXD)
- net ~{USB_{RST,1}}: now reaches U?.23 (PB4)
- net ~{USB_{RST,1}}: now also U?.65 (PJ2), U?.9 (~{RST})
- net ~{USB_{RST,2}}: now reaches U?.24 (PB5)
- net ~{USB_{RST,2}}: now also U?.66 (PJ3), U?.9 (~{RST})
- net ~{USB_{RST,3}}: now reaches U?.25 (PB6)
- net ~{USB_{RST,3}}: now also U?.67 (PJ4), U?.9 (~{RST})
- net LEDERROR: now reaches U?.26 (PB7)
- net LEDERROR: now also R?.1
- net PH7: now reaches U?.27 (PH7)
- net PH7: now also J?.18 (Pin_18)
- net USB_{1,TX}: now reaches U?.3 (PE1)
- net USB_{1,TX}: now also U?.64 (PJ1), U?.25 (RXD)
- net LEDBEAMON: now reaches U?.4 (PE2)
- net LEDBEAMON: now also R?.1
- net PL5: now reaches U?.40 (PL5)
- net PL5: now also J?.1 (Pin_1)
- net PL6: now reaches U?.41 (PL6)
- net PL6: now also J?.2 (Pin_2)
- net PL7: now reaches U?.42 (PL7)
- net PL7: now also J?.3 (Pin_3)
- net USB_{2,RX}: now reaches U?.45 (PD2)
- net USB_{2,RX}: now also U?.26 (TXD)
- net USB_{2,TX}: now reaches U?.46 (PD3)
- net USB_{2,TX}: now also U?.25 (RXD)
- net PD4: now reaches U?.47 (PD4)
- net PD4: now also J?.32 (Pin_32)
- net PD5: now reaches U?.48 (PD5)
- net PD5: now also J?.31 (Pin_31)
- net PD6: now reaches U?.49 (PD6)
- net PD6: now also J?.30 (Pin_30)
- net LEDFILON: now reaches U?.5 (PE3)
- net LEDFILON: now also R?.1
- net PD7: now reaches U?.50 (PD7)
- net PD7: now also J?.29 (Pin_29)
- net PG0: now reaches U?.51 (PG0)
- net PG0: now also J?.19 (Pin_19)
- net PH1: now reaches U?.52 (PG1)
- net PH1: now also J?.20 (Pin_20)
- net LEDHVON: now reaches U?.6 (PE4)
- net LEDHVON: now also R?.1
- net USB_{0,SUSPEND}: now reaches U?.68 (PJ5)
- net USB_{1,SUSPEND}: now reaches U?.69 (PJ6)
- net USB_{1,SUSPEND}: now also U?.12 (SUSPEND)
- net LEDWARNING: now reaches U?.7 (PE5)
- net LEDWARNING: now also R?.1
- net USB_{2,SUSPEND}: now reaches U?.79 (PJ7)
- net USB_{2,SUSPEND}: now also U?.12 (SUSPEND)
- net PK7: now reaches U?.82 (PK7)
- net PK7: now also J?.11 (Pin_11)
- net PK6: now reaches U?.83 (PK6)
- net PK6: now also J?.10 (Pin_10)
- net PK5: now reaches U?.84 (PK5)
- net PK5: now also J?.9 (Pin_9)
- net PK4: now reaches U?.85 (PK4)
- net PK4: now also J?.8 (Pin_8)
- net PK3: now reaches U?.86 (PK3)
- net PK3: now also J?.7 (Pin_7)
- net PK2: now reaches U?.87 (PK2)
- net PK2: now also J?.6 (Pin_6)
- net PK1: now reaches U?.88 (PK1)
- net PK1: now also J?.5 (Pin_5)
- net PK0: now reaches U?.89 (PK0)
- net PK0: now also J?.4 (Pin_4)
- net ILOCK: now reaches U?.9 (PE7)
- net ILOCK: now also J?.1 (Pin_1), R?.1
- net TDI: now reaches U?.90 (PF7)
- net TDI: now also J?.8 (Pin_8)
- net TDO: now reaches U?.91 (PF6)
- net TDO: now also J?.6 (Pin_6)
- net TMS: now reaches U?.92 (PF5)
- net TMS: now also J?.2 (Pin_2)
- net TCK: now reaches U?.93 (PF4)
- net TCK: now also J?.4 (Pin_4)
- net PF3: now reaches U?.94 (PF3)
- net PF3: now also J?.25 (Pin_25)
- net PF2: now reaches U?.95 (PF2)
- net PF2: now also J?.26 (Pin_26)
- net PF1: now reaches U?.96 (PF1)
- net PF1: now also J?.27 (Pin_27)
- net PF0: now reaches U?.97 (PF0)
- net PF0: now also J?.28 (Pin_28)
- new net: D?.2 (A), R?.2 (x11)
- new net: L?.2, U?.100 (AVCC)
- new net: R?.1, U?.18 (~{RXT}/GPIO.1) (x3)
- new net: R?.1, U?.19 (~{TXT}/GPIO.0) (x3)
- new net: D?.3 (K), J?.3 (D+), U?.4 (D+) (x3)
- new net: D?.2 (K), J?.2 (D-), U?.5 (D-) (x3)
- new net: C?.1, C?.1, U?.6 (VDD) (x3)
- new net: R?.2, R?.2, U?.8 (VBUS) (x3)
- new net: D?.4 (K), J?.1 (VBUS), R?.1 (x3)
- new net: J?.2 (Pin_2), R?.1
- new net: C?.2, C?.2 (x3)
- new net USB_{3,RX}: U?.26 (TXD)
- new net USB_{3,SUSPEND}: U?.12 (SUSPEND)
- new net USB_{3,TX}: U?.25 (RXD)
- new net ~{USB_{1,CTS}}: U?.23 (~{CTS})
- new net ~{USB_{1,DCD}}: U?.1 (~{DCD})
- new net ~{USB_{1,DSR}}: U?.27 (~{DSR})
- new net ~{USB_{1,DTR}}: JP?.1 (A), U?.28 (~{DTR})
- new net ~{USB_{1,RI}}: U?.2 (~{RI}/CLK)
- new net ~{USB_{1,RTS}}: U?.24 (~{RTS})
- new net ~{USB_{1,SUSPEND}}: R?.1, U?.11 (~{SUSPEND})
- new net ~{USB_{2,CTS}}: U?.23 (~{CTS})
- new net ~{USB_{2,DCD}}: U?.1 (~{DCD})
- new net ~{USB_{2,DSR}}: U?.27 (~{DSR})
- new net ~{USB_{2,DTR}}: JP?.1 (A), U?.28 (~{DTR})
- new net ~{USB_{2,RI}}: U?.2 (~{RI}/CLK)
- new net ~{USB_{2,RTS}}: U?.24 (~{RTS})
- new net ~{USB_{2,SUSPEND}}: R?.1, U?.11 (~{SUSPEND})
- new net ~{USB_{3,CTS}}: U?.23 (~{CTS})
- new net ~{USB_{3,DCD}}: U?.1 (~{DCD})
- new net ~{USB_{3,DSR}}: U?.27 (~{DSR})
- new net ~{USB_{3,DTR}}: JP?.1 (A), U?.28 (~{DTR})
- new net ~{USB_{3,RI}}: U?.2 (~{RI}/CLK)
- new net ~{USB_{3,RTS}}: U?.24 (~{RTS})
- new net ~{USB_{3,SUSPEND}}: R?.1, U?.11 (~{SUSPEND})
- no-connect marks 17 -> 42
Other:
- moved on the sheet: C?, D?, J?, R?, U?

Commit message: FInished Schematic, assigned footprints, added 230V PSU
Parts:
- added J10, J8, J9: Interlock, Connector_PinHeader_2.54mm:PinHeader_1x02_P2.54mm_Vertical, symbol Connector:Screw_Terminal_01x02
- added J?: Screw_Terminal_01x02, Connector_PinHeader_2.54mm:PinHeader_1x02_P2.54mm_Vertical, symbol Connector:Screw_Terminal_01x02
- added U?: AC-05-3, AC_05_3:AC-05-3, symbol AC053:AC-05-3
- C1, C10, C11, C12, C13, C14, C15, C16, C17, C18, C19, C2, C20, C21, C22, C23, C24, C25, C26, C27, C28, C29, C3, C30, C31, C32, C33, C34, C35, C36, C37, C38, C39, C4, C40, C41, C42, C5, C6, C7, C8, C9: renamed from C?; footprint (none) -> Capacitor_SMD:C_0805_2012Metric
- D1, D10, D11, D12, D13, D14, D15, D2, D3, D4, D5, D6: renamed from D?; footprint (none) -> LED_THT:LED_D3.0mm
- J1: renamed from J?; footprint (none) -> Connector_PinHeader_2.54mm:PinHeader_1x04_P2.54mm_Vertical
- J11: renamed from J?; footprint (none) -> Connector_PinHeader_2.54mm:PinHeader_2x04_P2.54mm_Vertical
- J12: renamed from J?; footprint (none) -> Connector_USB:USB_B_Lumberg_2411_02_Horizontal; FarnellNo (none) -> 3490505 (2401 06)
- J13, J14: renamed from J?; footprint (none) -> Connector_USB:USB_B_Lumberg_2411_02_Horizontal
- J15: renamed from J?; footprint (none) -> Connector_Dsub:DSUB-15_Female_Horizontal_P2.77x2.84mm_EdgePinOffset9.90mm_Housed_MountingHolesOffset11.32mm; FarnellNo (none) -> 3817870
- J16, J17, J18: renamed from J?; footprint (none) -> Connector_Dsub:DSUB-15_Female_Horizontal_P2.77x2.84mm_EdgePinOffset9.90mm_Housed_MountingHolesOffset11.32mm
- J2: renamed from J?; footprint (none) -> Connector_PinHeader_2.54mm:PinHeader_1x02_P2.54mm_Vertical
- J3, J6, J7: renamed from J?; footprint (none) -> Connector_PinHeader_2.54mm:PinHeader_2x16_P2.54mm_Vertical
- J4: renamed from J?; footprint (none) -> Connector_PinSocket_2.54mm:PinSocket_2x03_P2.54mm_Vertical
- J5: renamed from J?; footprint (none) -> Connector_PinSocket_2.54mm:PinSocket_2x05_P2.54mm_Vertical
- JP1, JP2, JP3: renamed from JP?; footprint (none) -> Connector_PinSocket_2.54mm:PinSocket_1x02_P2.54mm_Vertical
- L1: renamed from L?; footprint (none) -> Inductor_SMD:L_1206_3216Metric
- R1, R10, R11, R12, R13, R14, R15, R16, R17, R18, R19, R2, R20, R21, R22, R23, R24, R25, R26, R27, R28, R29, R3, R30, R31, R32, R33, R34, R35, R36, R37, R38, R39, R4, R40, R41, R42, R43, R44, R45, R46, R47, R48, R49, R5, R50, R51, R52, R53, R54, R55, R56, R57, R58, R59, R6, R60, R61, R62, R63, R64, R65, R66, R67, R68, R69, R7, R70, R71, R72, R73, R74, R75, R76, R77, R78, R79, R8, R80, R81, R82, R83, R84, R85, R86, R87, R88, R89, R9, R90: renamed from R?; footprint (none) -> Resistor_SMD:R_0805_2012Metric
- U10, U11, U12, U13, U14, U7, U8, U9: renamed from U?; footprint (none) -> Package_DIP:DIP-8_W7.62mm
- U2, U3: renamed from U?; footprint (none) -> Package_SO:SOIC-14_3.9x8.7mm_P1.27mm
- Y1: renamed from Y?; footprint (none) -> Connector_PinSocket_2.54mm:PinSocket_1x03_P2.54mm_Vertical
- gave numbers to parts that had none: 15
Connections:
- net +5V: now also U?.3 (+5V)
- net GND: now also U?.4 (V-)
- net USB_{1,RX}: now also J8.2 (Pin_2)
- net USB_{1,TX}: now also J8.1 (Pin_1)
- net USB_{2,RX}: now also J9.2 (Pin_2)
- net USB_{2,TX}: now also J9.1 (Pin_1)
- net USB_{3,RX}: now also J10.2 (Pin_2)
- net USB_{3,TX}: now also J10.1 (Pin_1)
- new net: J?.1 (Pin_1), U?.2 (AC/N)
- new net: J?.2 (Pin_2), U?.1 (AC/L)

Commit message: Continue place and route, minor fixes
Parts:
- J10: value Interlock -> USART3
- J8: value Interlock -> USART1
- J9: value Interlock -> USART2
- gave numbers to parts that had none: 2
Connections:
- net CC_{1}: no longer J16.1, J17.1, J18.1, R57.2, R61.2, R67.2
- net CV_{1}: no longer J16.2, J17.2, J18.2, R81.2, R84.2, R88.2
- net I_{mon,2}: now also J17.3, R85.2
- net I_{mon,3}: now also J16.3, R82.2
- net I_{mon,4}: now also J18.3, R89.2
- net I_{mon}: no longer J16.3, J17.3, J18.3, R82.2, R85.2, R89.2
- net I_{set,1}: no longer J16.15 (P15), J17.15 (P15), J18.15 (P15), R46.2, R48.2, R50.2, U10.7, U8.7, U9.7
- net POL_{set,1}: no longer J16.7, J17.7, J18.7, U17.4, U19.4, U21.4
- net POL_{set,2}: now also J17.7, U19.4
- net POL_{set,3}: now also J16.7, U17.4
- net POL_{set,4}: now also J18.7, U21.4
- net UNIT_{ON,1}: no longer J16.12 (P12), J17.12 (P12), J18.12 (P12), U18.4, U20.4, U22.4
- net UNIT_{ON,2}: now also J17.12 (P12), U20.4
- net UNIT_{ON,3}: now also J16.12 (P12), U18.4
- net UNIT_{ON,4}: now also J18.12 (P12), U22.4
- net V_{mon,2}: now also J17.11 (P111), R86.2
- net V_{mon,3}: now also J16.11 (P111), R83.2
- net V_{mon,4}: now also J18.11 (P111), R90.2
- net V_{mon}: no longer J16.11 (P111), J17.11 (P111), J18.11 (P111), R83.2, R86.2, R90.2
- net V_{set,1}: no longer J16.8, J17.8, J18.8, R45.2, R47.2, R49.2, U10.1, U8.1, U9.1
- net ~{USB_{RST,1}}: no longer U1.65 (PJ2)
- net ~{USB_{RST,2}}: no longer U1.66 (PJ3)
- net ~{USB_{RST,3}}: no longer U1.67 (PJ4)
- new net CC_{2}: J17.1, R61.2
- new net CC_{3}: J16.1, R57.2
- new net CC_{4}: J18.1, R67.2
- new net CV_{2}: J17.2, R84.2
- new net CV_{3}: J16.2, R81.2
- new net CV_{4}: J18.2, R88.2
- new net I_{set,2}: J17.15 (P15), R48.2, U9.7
- new net I_{set,3}: J16.15 (P15), R46.2, U8.7
- new net I_{set,4}: J18.15 (P15), R50.2, U10.7
- new net V_{set,2}: J17.8, R47.2, U9.1
- new net V_{set,3}: J16.8, R45.2, U8.1
- new net V_{set,4}: J18.8, R49.2, U10.1
